Commit message: support visual u-arm in rerun

File: assets/robots/uarm_config2/uarm_config2_leader.urdf (robot description, URDF)
Before this commit: robot uarm_config2_leader, 7 links, 6 joints
Joints:
- joint joint1: axis 0.000000 0.000000 1.000000 -> 0.3695929294 -0.9283029711 -0.0406775179; origin xyz=0.114500 0.201100 0.125600 rpy=0 0 0 -> xyz=0.1207304713 0.2031548637 0.1353154913 rpy=0 0 0
- joint joint2: axis 0.615551 0.764790 0.190244 -> 0.9104260564 0.3705284163 -0.1839377299; origin xyz=0.015100 0.048800 0.014900 rpy=0 0 0 -> xyz=0.0033769596 0.0532948105 -0.0088079311 rpy=0 0 0
- joint joint3: axis 0.615551 0.764790 0.190244 -> 0.9104257971 0.3705305088 -0.1839347981; origin xyz=-0.052300 0.070900 -0.115800 rpy=0 0 0 -> xyz=-0.0516695545 0.0745506831 -0.1053254329 rpy=0 0 0
- joint joint4: axis 0.615551 0.764790 0.190244 -> 0.9104241205 0.3705338696 -0.1839363266; origin xyz=-0.053200 0.026600 0.065200 rpy=0 0 0 -> xyz=-0.0489368402 0.0226440259 0.0783323102 rpy=0 0 0
- joint joint5: axis 0.678176 -0.637002 0.366478 -> 0.2263241889 -0.0739567991 0.9712403170; origin xyz=0.048600 -0.002600 0.065200 rpy=0 0 0 -> xyz=0.0407671249 -0.0023330755 0.0580462147 rpy=0 0 0
- joint joint6: axis 0.233403 -0.495747 0.836515 -> -0.4831945686 0.8572534066 0.1778752532; origin xyz=-0.010700 0.023300 0.060300 rpy=0 0 0 -> xyz=0.0022162481 0.0173025380 0.0675447238 rpy=0 0 0

Commit message: support visual u-arm in rerun

File: assets/robots/uarm_config2/uarm_config2_leader.urdf (robot description, URDF)
Before this commit: robot uarm_config2_leader, 7 links, 6 joints
Joints:
- joint joint1: axis 0.3695929294 -0.9283029711 -0.0406775179 -> -0.3695929294 0.9283029711 0.0406775179
- joint joint4: axis 0.9104241205 0.3705338696 -0.1839363266 -> -0.9104241205 -0.3705338696 0.1839363266

Commit message: support visual u-arm in rerun

File: assets/robots/uarm_config2/uarm_config2_leader.urdf (robot description, URDF)
Before this commit: robot uarm_config2_leader, 7 links, 6 joints
Joints:
- joint joint1: origin xyz=0.1207304713 0.2031548637 0.1353154913 rpy=0 0 0 -> xyz=0.1207304713 0.2031548637 0.1353154913 rpy=0.065655549893 -0.161673104370 -0.012438471256
- joint joint2: origin xyz=0.0033769596 0.0532948105 -0.0088079311 rpy=0 0 0 -> xyz=0.0033769596 0.0532948105 -0.0088079311 rpy=0.883730524893 0.384319890433 -0.007360790781
- joint joint3: origin xyz=-0.0516695545 0.0745506831 -0.1053254329 rpy=0 0 0 -> xyz=-0.0516695545 0.0745506831 -0.1053254329 rpy=-2.514047085138 0.127563143479 0.814471975469
